Commit message: Collect data 2.5x faster, and use real PBR materials and a table mesh
Data rate. Episode time 45 s -> 18 s from three measured changes:
  - real_time_factor 1.0 -> 0, so physics runs unthrottled rather than pacing
    to wall-clock. Everything downstream uses use_sim_time and follows /clock,
    so the recorded data is identical, just collected sooner
  - MoveIt velocity/acceleration scaling 0.25 -> 0.6. Most of an episode is the
    arm travelling between waypoints, so this is the biggest single lever
  - cameras 640x480 -> 320x240 (launch argument). The policy downsamples to
    224x224 anyway, so the extra pixels were discarded work. Camera rate went
    19.8 -> 39 Hz

collect_parallel.sh runs N independent simulations at once. Each worker needs
its own ROS_DOMAIN_ID *and* its own GZ_PARTITION: the domain id separates the
DDS network, but Gazebo's transport discovery ignores it, so without a
partition two simulations fight over world and service names. merge_demos.py
folds the workers into one dataset, renumbering as it copies since every worker
numbers from zero, and recording provenance. Verified with 2 workers x 2
episodes merged to 4 with correct indices and tasks.

Appearance. Real CC0 PBR sets from ambientcg.com (Wood062, Concrete034,
Metal032, Plaster001) replace the procedural stand-ins, and the worktop is now
a generated workbench.stl with apron, chamfered lip and stretcher shelf.
Collision remains a box. Textures are git-ignored and fetched by
materials/fetch_ambientcg.sh, so the repo carries no third-party binaries and
still loads without them.

NormalGL, not NormalDX: Ogre2 expects the OpenGL convention. The DirectX
variant has the green channel inverted and lights surfaces inside-out.

Fixed: meshes/ was missing from the CMakeLists install list, so the mesh URI
could not be resolved and the entire world failed to load.

Co-Authored-By: Claude Opus 5 <noreply@anthropic.com>

File: src/groot_arm_description/urdf/groot_arm.urdf.xacro (robot description, xacro)
@@ -31,4 +31,11 @@
   <xacro:property name="pedestal_height" value="0.6"/>
   <xacro:property name="gripper_stroke" value="0.04"/>
+  <!-- The policy downsamples to 224x224 regardless, so rendering 640x480 is
+       mostly wasted GPU. 320x240 stays above that and roughly halves the
+       render cost. Raise it if you want nicer recordings to look at. -->
+  <xacro:arg name="camera_width" default="320"/>
+  <xacro:arg name="camera_height" default="240"/>
+  <xacro:property name="camera_width" value="$(arg camera_width)"/>
+  <xacro:property name="camera_height" value="$(arg camera_height)"/>
   <!-- =========================== world =========================== -->
   <link name="world"/>
@@ -84,5 +91,5 @@
        camera. Gazebo's optical axis is +x. -->
   <xacro:rgb_camera name="wrist_camera" parent="${tf_prefix}gripper_base_link"
-                    width="640" height="480" hfov="1.4">
+                    width="${camera_width}" height="${camera_height}" hfov="1.4">
     <origin xyz="0.05 0 0.025" rpy="0 ${-2.2865} 0"/>
   </xacro:rgb_camera>
@@ -114,5 +121,5 @@
        field. rpy derived from that sight line; see README if you move the mast. -->
   <xacro:rgb_camera name="scene_camera" parent="camera_mast_link"
-                    width="640" height="480" hfov="1.25">
+                    width="${camera_width}" height="${camera_height}" hfov="1.25">
     <origin xyz="0 0 1.1" rpy="0 0.7000 -0.7247"/>
   </xacro:rgb_camera>
